Commit message: updated robot urdf and pybullet environment

File: software/simulation/urdf/robotic_arm.urdf (robot description, URDF)
Before this commit: robot robotic_arm, 4 links, 3 joints
Links:
- removed link base_link
- removed link link1
- removed link link2
- removed link link3
- added link baseLink, mass .5; collision box size=0.005 0.125 0.105; visual box size=0.026 0.026 0.150
- added link linkA, mass .3; collision box size=0.07 0.055 0.11; visual box size=0.026 0.026 0.150
- added link linkA10, mass .1; collision box size=0.005 0.02 0.17; visual box size=0.026 0.026 0.150
- added link linkA9, mass .1; collision box size=0.005 0.02 0.18; visual box size=0.026 0.026 0.150
- added link linkB, mass .1; collision box size=0.036 0.036 0.150; visual box size=0.005 0.185 0.05
- added link linkC, mass .1; collision box size=0.026 0.026 0.21; visual box size=0.005 0.22 0.06
- added link linkC2, mass .1; collision box size=0.026 0.026 0.150; visual box size=0.026 0.026 0.150
- added link linkD, mass .1; collision box size=0.02 0.08 0.005; visual box size=0.005 0.045 0.037
- added link motorA, mass .1; collision cylinder length=0.03 radius=0.02; visual cylinder length=0.03 radius=0.02
- added link motorB, mass .1; collision cylinder length=0.03 radius=0.02; visual cylinder length=0.03 radius=0.02
Joints:
- removed joint joint1
- removed joint joint2
- removed joint joint3
- added joint joint_baseLink_childA: type continuous, parent baseLink, child linkA, origin xyz=0.0 0.0 0.06, axis 0 0 1
- added joint joint_linkAlinkA9: type continuous, parent linkA, child linkA9, origin xyz=0 -0.026 0.054, axis 1 0 0
- added joint joint_linkAlinkB: type continuous, parent linkA, child linkB, origin xyz=0 0.0 0.04, axis 1 0 0
- added joint joint_linkAmotorA: type continuous, parent linkA, child motorA, origin xyz=0.05 0.0 0.03, axis 1 0 0
- added joint joint_linkAmotorB: type continuous, parent linkA, child motorB, origin xyz=-0.05 0.0 0.03, axis -1 0 0
- added joint joint_linkBlinkC: type continuous, parent linkB, child linkC, origin xyz=0.0 0.0 0.150, axis 1 0 0
- added joint joint_linkBlinkC2: type continuous, parent linkB, child linkC2, origin xyz=0.0 0.0 0.150, axis 1 0 0
- added joint joint_linkC2linkA10: type continuous, parent linkC2, child linkA10, origin xyz=0 0.026 0.014, axis 1 0 0
- added joint joint_linkClinkD: type continuous, parent linkC, child linkD, origin xyz=0.0 0.00 0.160, axis 1 0 0
