Commit message: robot can track a point in simulation

File: software/simulation/urdf/simple_arm.urdf (robot description, URDF)
Before this commit: robot simple__arm, 4 links, 3 joints
Links:
- added link tool_link, mass 0.01; collision sphere radius=0.005; visual sphere radius=0.005
- link link3: geometry collision cylinder length=0.15 radius=0.01; visual cylinder length=0.15 radius=0.01
Joints:
- added joint joint4: type fixed, parent link3, child tool_link, origin xyz=0 0 0.15, axis 0 0 0
